Commit message: update!

File: nextage_fillie_open_description/urdf/FillieOpen.urdf (robot description, URDF)
Before this commit: robot NEXTAGE, 16 links, 15 joints
Links:
- added link world
- link WAIST: mass None -> 10000
Joints:
- added joint fixed: type fixed, parent world, child WAIST
- joint CHEST_JOINT0: limit lower=-3.141592654 upper=3.141592654 effort=100 velocity=1.0 -> lower=-3.141592654 upper=3.141592654 effort=100.0 velocity=1.0
- joint HEAD_JOINT0: limit lower=-1.570796327 upper=1.570796327 effort=100 velocity=1.0 -> lower=-1.570796327 upper=1.570796327 effort=100.0 velocity=1.0
- joint HEAD_JOINT1: limit lower=-0.401425728 upper=1.308996939 effort=100 velocity=1.0 -> lower=-0.401425728 upper=1.308996939 effort=100.0 velocity=1.0
- joint LARM_JOINT0: limit lower=-1.570796327 upper=1.570796327 effort=150 velocity=1.0 -> lower=-1.570796327 upper=1.570796327 effort=150.0 velocity=1.0; origin xyz=0.0 0.155 0.520 rpy=-0.26179938779914941 0 0 -> xyz=0.0 0.155 0.520 rpy=-0.26179938779914941 0.0 0.0
- joint LARM_JOINT1: limit lower=-2.443460953 upper=1.570796327 effort=150 velocity=1.0 -> lower=-2.443460953 upper=1.570796327 effort=150.0 velocity=1.0; origin xyz=0 0.0 0.0 rpy=0 0 0 -> xyz=0.0 0.0 0.0 rpy=0.0 0.0 0.0
- joint LARM_JOINT2: limit lower=-1.221730476 upper=1.570796327 effort=150 velocity=1.0 -> lower=-1.221730476 upper=1.570796327 effort=150.0 velocity=1.0
- joint LARM_JOINT3: limit lower=-3.141592654 upper=1.745329252 effort=150 velocity=1.0 -> lower=-3.141592654 upper=1.745329252 effort=150.0 velocity=1.0
- joint LARM_JOINT4: limit lower=-1.570796327 upper=1.570796327 effort=150 velocity=1.0 -> lower=-1.570796327 upper=1.570796327 effort=150.0 velocity=1.0
- joint LARM_JOINT5: limit lower=-2.9670597283903604 upper=2.9670597283903604 effort=150 velocity=1.0 -> lower=-2.9670597283903604 upper=2.9670597283903604 effort=150.0 velocity=1.0
- joint RARM_JOINT0: limit lower=-1.570796327 upper=1.570796327 effort=150 velocity=1.0 -> lower=-1.570796327 upper=1.570796327 effort=150.0 velocity=1.0
- joint RARM_JOINT1: limit lower=-2.443460953 upper=1.570796327 effort=150 velocity=1.0 -> lower=-2.443460953 upper=1.570796327 effort=150.0 velocity=1.0
- joint RARM_JOINT2: limit lower=-1.221730476 upper=1.570796327 effort=150 velocity=1.0 -> lower=-1.221730476 upper=1.570796327 effort=150.0 velocity=1.0
- joint RARM_JOINT3: limit lower=-1.745329252 upper=3.141592654 effort=150 velocity=1.0 -> lower=-1.745329252 upper=3.141592654 effort=150.0 velocity=1.0
- joint RARM_JOINT4: limit lower=-1.570796327 upper=1.570796327 effort=150 velocity=1.0 -> lower=-1.570796327 upper=1.570796327 effort=150.0 velocity=1.0
- joint RARM_JOINT5: limit lower=-2.9670597283903604 upper=2.9670597283903604 effort=150 velocity=1.0 -> lower=-2.9670597283903604 upper=2.9670597283903604 effort=150.0 velocity=1.0

File: nextage_fillie_open_description/urdf/nextage_fillie_open_gz.xacro (robot description, xacro)
@@ -2,32 +2,38 @@
 <robot name="FillieOpen"
        xmlns:xacro="http://www.ros.org/wiki/xacro">
-  <xacro:include filename="$(find nextage_fillie_open_description)/urdf/FillieOpen.urdf" />
-  <xacro:include filename="$(find nextage_fillie_open_description)/urdf/nextage_fillie_open_gz_camera.xacro" />
-  <xacro:property name="M_PI" value="3.1415926535897931" />
-  <xacro:property name="jnt_head_camera_displacement_x" value="0.0175" />
-  <xacro:property name="jnt_head_camera_displacement_y" value="0.0725" />
-  <xacro:property name="jnt_head_camera_displacement_z" value="0.105" />
-  <xacro:property name="jnt_head_camera_rot_y" value="0.25" />
-  <xacro:property name="link_head_camera_rot_z" value="0.05" />
-  <!-- NOTE: The poses of headmount cameras are NOT precisely adjusted to
-             the 3D model nor the actual hardware config. These configs
-             are meant for a rapid prototyping only. If you need precise
-             configuration, please go ahead modify the following, then
-             (if possible) send a patch to https://github.com/tork-a/rtmros_nextage/pulls
-             so that other developers and users can use (and possible improve).
-  -->
-  <xacro:camera_joint_link_gzplugin
-         camera_name="CAMERA_HEAD_L" link_parent="HEAD_JOINT1_Link"
-         jnt_displacement_x="${jnt_head_camera_displacement_x}" jnt_displacement_y="${jnt_head_camera_displacement_y}" jnt_displacement_z="${jnt_head_camera_displacement_z}"
-         jnt_rotation_x="0" jnt_rotation_y="${jnt_head_camera_rot_y}" jnt_rotation_z="0"
-         link_displacement_x="0.0325" link_displacement_y="0" link_displacement_z="0"
-         link_rotation_x="0" link_rotation_y="${M_PI/2}" link_rotation_z="-${link_head_camera_rot_z}" />
-  <xacro:camera_joint_link_gzplugin
-         camera_name="CAMERA_HEAD_R" link_parent="HEAD_JOINT1_Link"
-         jnt_displacement_x="${jnt_head_camera_displacement_x}" jnt_displacement_y="-${jnt_head_camera_displacement_y}" jnt_displacement_z="${jnt_head_camera_displacement_z}"
-         jnt_rotation_x="0" jnt_rotation_y="${jnt_head_camera_rot_y}" jnt_rotation_z="0"
-         link_displacement_x="0.0325" link_displacement_y="0" link_displacement_z="0"
-         link_rotation_x="0" link_rotation_y="${M_PI/2}" link_rotation_z="${link_head_camera_rot_z}" />
-  <!-- TODO hand cameras can be added here with the very similar code as
-            headmount cameras. -->
+       <!-- <xacro:include filename="$(find nextage_fillie_open_description)/urdf/FillieOpen.urdf" /> -->
+       <xacro:include filename="$(find nextage_fillie_open_description)/urdf/nextage_fillie_open_gz_camera.xacro" />
+       <xacro:property name="M_PI" value="3.1415926535897931" />
+       <xacro:property name="jnt_head_camera_displacement_x" value="0.0175" />
+       <xacro:property name="jnt_head_camera_displacement_y" value="0.0725" />
+       <xacro:property name="jnt_head_camera_displacement_z" value="0.105" />
+       <xacro:property name="jnt_head_camera_rot_y" value="0.25" />
+       <xacro:property name="link_head_camera_rot_z" value="0.05" />
+       <!-- NOTE: The poses of headmount cameras are NOT precisely adjusted to
+              the 3D model nor the actual hardware config. These configs
+              are meant for a rapid prototyping only. If you need precise
+              configuration, please go ahead modify the following, then
+              (if possible) send a patch to https://github.com/tork-a/rtmros_nextage/pulls
+              so that other developers and users can use (and possible improve).
+       -->
+       <!-- TODO hand cameras can be added here with the very similar code as
+       headmount cameras. -->
+       <xacro:macro name="joint_transmission" params="name reduction offset_value">
+              <transmission name="${name}_trans">
+                     <plugin>transmission_interface/SimpleTransmission</plugin>
+                     <actuator name="${name}_actuator" role="actuator1"/>
+                     <joint name="${name}" role="joint1" >
+                            <offset>${offset_value}</offset>
+                            <mechanicalReduction>${reduction}</mechanicalReduction>
+                     </joint>
+              </transmission>
+       </xacro:macro>
+       <xacro:macro name="ros2_control_joint" params="name reduction offset_value" >
+              <joint name="${name}">
+                     <command_interface name="position" />
+                     <state_interface name="position" />
+                     <state_interface name="velocity" />
+              </joint>
+              <xacro:joint_transmission name="${name}" reduction="1" offset_value="${offset_value}" />
+       </xacro:macro>
 </robot>

File: nextage_fillie_open_description/urdf/nextage_fillie_open_gz_camera.xacro (robot description, xacro)
@@ -24,5 +24,5 @@
 					<cylinder length="0.01" radius="0.015" />
 				</geometry>
-				<material name="blue" />
+				<material name="Blue" />
 			</visual>
 			<inertial>
@@ -56,5 +56,5 @@
 					</noise>
 				</camera>
-				<plugin name="camera_controller" filename="libgazebo_ros_camera.so">
+				<plugin name="camera_controller" filename="libgazebo_ros2_camera.so">
 					<alwaysOn>true</alwaysOn>
 					<updateRate>0.0</updateRate>
